File: Starter-Keyboard.kicad_sch (KiCad schematic)
At the start: 0 parts

Commit message: updated keyboard, started work on pcb
Parts:
- added D1, D10, D11, D12, D13, D14, D18, D19, D2, D25, D26, D27, D28, D29, D3, D4, D5, D6, D7, D8: 1N4148, Diode_THT:D_DO-35_SOD27_P7.62mm_Horizontal, symbol Diode:1N4148
- added J1: Conn_01x02_Socket, Connector_JST:JST_PH_S2B-PH-SM4-TB_1x02-1MP_P2.00mm_Horizontal, symbol Connector:Conn_01x02_Socket
- added SW1, SW10, SW11, SW12, SW15, SW16, SW18, SW19, SW2, SW25, SW26, SW27, SW28, SW29, SW3, SW4, SW5, SW6, SW7, SW8: SW_Push, MX_V2:Gateron-KS33-Hotswap-1U, symbol Switch:SW_Push
- added SW13: RotaryEncoder, temp:XDCR_PEC11R-4220F-S0024, symbol Device:RotaryEncoder
- added SW14: SW_SPDT, Button_Switch_SMD:SW_SPDT_PCM12, symbol Switch:SW_SPDT
- added U2: XIAO-MG24-DIP, Seeed_Studio_XIAO_Series:XIAO-MG24-DIP, symbol Seeed_Studio_XIAO_Series:XIAO-MG24-DIP
Connections:
- new net: J1.1 (Pin_1), SW14.1 (A)
- new net: D7.2 (A), SW7.2
- new net: D5.2 (A), SW5.2
- new net: D1.2 (A), SW1.2
- new net: D19.2 (A), SW19.2
- new net: D14.2 (A), SW16.2
- new net: D29.2 (A), SW29.2
- new net: D3.2 (A), SW3.2
- new net: D18.2 (A), SW18.2
- new net: D27.2 (A), SW27.2
- new net: D8.2 (A), SW8.2
- new net: D10.2 (A), SW10.2
- new net: D4.2 (A), SW4.2
- new net: D11.2 (A), SW11.2
- new net: D12.2 (A), SW12.2
- new net: D2.2 (A), SW2.2
- new net: D6.2 (A), SW6.2
- new net: D25.2 (A), SW25.2
- new net: D26.2 (A), SW26.2
- new net: D28.2 (A), SW28.2
- new net: D13.2 (A), SW15.2
- new net GND: SW13.C, U2.13 (GND)
- new net bat +: SW14.2 (B)
- new net bat -: J1.2 (Pin_2)
- new net col 1: SW25.1, SW26.1, SW27.1, SW28.1, SW29.1, U2.7 (PC06_A6_D6_TX)
- new net col 2: SW1.1, SW10.1, SW16.1, SW4.1, SW7.1, U2.11 (PA05_A10_D10_MOSI)
- new net col 3: SW11.1, SW18.1, SW2.1, SW5.1, SW8.1, U2.10 (PA04_A9_D9_MISO)
- new net col 4: SW12.1, SW15.1, SW19.1, SW3.1, SW6.1, U2.9 (PA03_A8_D8_SCK)
- new net pin A: SW13.A, U2.6 (PC05_A5_D5_SCL)
- new net pin B: SW13.B, U2.8 (PC07_A7_D7_RX)
- new net row 1: D1.1 (K), D2.1 (K), D25.1 (K), D3.1 (K), U2.1 (PC00_A0_D0)
- new net row 2: D26.1 (K), D4.1 (K), D5.1 (K), D6.1 (K), U2.2 (PC01_A1_D1)
- new net row 3: D13.1 (K), D27.1 (K), D7.1 (K), D8.1 (K), U2.3 (PC02_A2_D2)
- new net row 4: D10.1 (K), D11.1 (K), D12.1 (K), D28.1 (K), U2.4 (PC03_A3_D3)
- new net row 5: D14.1 (K), D18.1 (K), D19.1 (K), D29.1 (K), U2.5 (PC04_A4_D4_SDA)
- no-connect marks 0 -> 3
